File: power_sch.kicad_sch (KiCad schematic)
At the start: 9 parts, among them J1 12V Terminal Block, J2 Barrel_Jack, J3 USB_A, SW1 SW_DPST_x2

Commit message: Schematic in state of received unit.  Will branch from here.
Parts:
- removed J1: 12V Terminal Block, symbol Connector:Screw_Terminal_01x04
- added TB1: ~, symbol Project Library:Terminal_Block_4
Connections:
- net 12V DC: now also TB1.1B, TB1.2B; no longer SW1.2 (B)
- net 12V GND: now also TB1.3B, TB1.4B
- new net: SW1.2 (B), TB1.2A
Changed lines of the file:
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@@
     (title "Power")
   )
-  (junction (at 227.33 88.9) (diameter 0) (color 0 0 0 0)
-  )
   (junction (at 137.16 115.57) (diameter 0) (color 0 0 0 0)
   )
@@
   (junction (at 113.03 95.25) (diameter 0) (color 0 0 0 0)
   )
-  (junction (at 234.95 88.9) (diameter 0) (color 0 0 0 0)
+  (junction (at 234.95 76.2) (diameter 0) (color 0 0 0 0)
   )
   (junction (at 113.03 85.09) (diameter 0) (color 0 0 0 0)
   )
-  (junction (at 229.87 88.9) (diameter 0) (color 0 0 0 0)
-  )
   (junction (at 234.95 95.25) (diameter 0) (color 0 0 0 0)
+  )
+  (junction (at 234.95 81.28) (diameter 0) (color 0 0 0 0)
+  )
+  (junction (at 234.95 78.74) (diameter 0) (color 0 0 0 0)
+  )
+  (junction (at 234.95 83.82) (diameter 0) (color 0 0 0 0)
   )
   (no_connect (at 304.8 115.57))
   (no_connect (at 304.8 113.03))
-  (wire (pts (xy 210.82 92.71) (xy 229.87 92.71))
-    (stroke (width 0) (type default))
-  )
   (wire (pts (xy 154.94 104.14) (xy 163.83 104.14))
     (stroke (width 0) (type default))
@@
     (stroke (width 0) (type default))
   )
-  (wire (pts (xy 234.95 95.25) (xy 234.95 88.9))
-    (stroke (width 0) (type default))
-  )
   (wire (pts (xy 290.83 107.95) (xy 304.8 107.95))
     (stroke (width 0) (type default))
@@
     (stroke (width 0) (type default))
   )
+  (wire (pts (xy 234.95 95.25) (xy 234.95 101.6))
+    (stroke (width 0) (type default))
+  )
   (wire (pts (xy 194.31 92.71) (xy 200.66 92.71))
     (stroke (width 0) (type default))
   )
+  (wire (pts (xy 222.25 78.74) (xy 227.33 78.74))
+    (stroke (width 0) (type default))
+  )
   (wire (pts (xy 104.14 88.9) (xy 104.14 85.09))
     (stroke (width 0) (type default))
@@
     (stroke (width 0) (type default))
   )
-  (wire (pts (xy 234.95 88.9) (xy 240.03 88.9))
-    (stroke (width 0) (type default))
-  )
-  (wire (pts (xy 227.33 96.52) (xy 227.33 88.9))
+  (wire (pts (xy 234.95 81.28) (xy 240.03 81.28))
+    (stroke (width 0) (type default))
+  )
+  (wire (pts (xy 234.95 83.82) (xy 234.95 95.25))
     (stroke (width 0) (type default))
   )
@@
     (stroke (width 0) (type default))
   )
+  (wire (pts (xy 234.95 76.2) (xy 240.03 76.2))
+    (stroke (width 0) (type default))
+  )
   (wire (pts (xy 313.69 123.19) (xy 314.96 123.19))
     (stroke (width 0) (type default))
@@
     (stroke (width 0) (type default))
   )
-  (wire (pts (xy 229.87 92.71) (xy 229.87 88.9))
-    (stroke (width 0) (type default))
-  )
   (wire (pts (xy 154.94 115.57) (xy 137.16 115.57))
     (stroke (width 0) (type default))
   )
-  (wire (pts (xy 262.89 96.52) (xy 227.33 96.52))
-    (stroke (width 0) (type default))
-  )
-  (wire (pts (xy 227.33 88.9) (xy 229.87 88.9))
+  (wire (pts (xy 222.25 92.71) (xy 222.25 78.74))
+    (stroke (width 0) (type default))
+  )
+  (wire (pts (xy 210.82 92.71) (xy 222.25 92.71))
+    (stroke (width 0) (type default))
+  )
+  (wire (pts (xy 234.95 76.2) (xy 234.95 78.74))
     (stroke (width 0) (type default))
   )
@@
     (stroke (width 0) (type default))
   )
+  (wire (pts (xy 234.95 81.28) (xy 234.95 83.82))
+    (stroke (width 0) (type default))
+  )
   (wire (pts (xy 113.03 85.09) (xy 163.83 85.09))
     (stroke (width 0) (type default))
@@
     (stroke (width 0) (type default))
   )
+  (wire (pts (xy 262.89 96.52) (xy 251.46 96.52))
+    (stroke (width 0) (type default))
+  )
   (wire (pts (xy 312.42 124.46) (xy 312.42 123.19))
     (stroke (width 0) (type default))
   )
-  (wire (pts (xy 234.95 101.6) (xy 234.95 95.25))
-    (stroke (width 0) (type default))
-  )
   (wire (pts (xy 163.83 85.09) (xy 163.83 92.71))
     (stroke (width 0) (type default))
@@
     (stroke (width 0) (type default))
   )
-  (wire (pts (xy 222.25 88.9) (xy 227.33 88.9))
-    (stroke (width 0) (type default))
-  )
-  (wire (pts (xy 232.41 88.9) (xy 234.95 88.9))
+  (wire (pts (xy 251.46 96.52) (xy 251.46 78.74))
     (stroke (width 0) (type default))
   )
@@
     (stroke (width 0) (type default))
   )
+  (wire (pts (xy 251.46 78.74) (xy 234.95 78.74))
+    (stroke (width 0) (type default))
+  )
   (wire (pts (xy 113.03 107.95) (xy 113.03 101.6))
     (stroke (width 0) (type default))
@@
     )
   )
-  (global_label "12V DC" (shape passive) (at 222.25 88.9 180) (fields_autoplaced)
-    (effects (font (size 1.27 1.27)) (justify right))
-    (property "Intersheetrefs" "${INTERSHEET_REFS}" (at 213.3609 88.9 0)
-      (effects (font (size 1.27 1.27)) (justify right) hide)
-    )
-  )
   (global_label "5V GND" (shape passive) (at 287.02 97.79 0) (fields_autoplaced)
     (effects (font (size 1.27 1.27)) (justify left))
@@
     )
   )
-  (global_label "12V GND" (shape passive) (at 240.03 88.9 0) (fields_autoplaced)
-    (effects (font (size 1.27 1.27)) (justify left))
-    (property "Intersheetrefs" "${INTERSHEET_REFS}" (at 250.2496 88.9 0)
-      (effects (font (size 1.27 1.27)) (justify left) hide)
+  (global_label "12V DC" (shape passive) (at 240.03 76.2 0) (fields_autoplaced)
+    (effects (font (size 1.27 1.27)) (justify left))
+    (property "Intersheetrefs" "${INTERSHEET_REFS}" (at 248.9191 76.2 0)
+      (effects (font (size 1.27 1.27)) (justify left) hide)
+    )
+  )
+  (global_label "12V GND" (shape passive) (at 240.03 81.28 0) (fields_autoplaced)
+    (effects (font (size 1.27 1.27)) (justify left))
+    (property "Intersheetrefs" "${INTERSHEET_REFS}" (at 250.2496 81.28 0)
+      (effects (font (size 1.27 1.27)) (justify left) hide)
+    )
+  )
+  (symbol (lib_id "Project Library:Terminal_Block_4") (at 231.14 73.66 0) (unit 1)
+    (in_bom yes) (on_board yes) (dnp no) (fields_autoplaced)
+    (property "Reference" "TB1" (at 231.14 72.39 0)
+      (effects (font (size 1.27 1.27)))
+    )
+    (property "Value" "~" (at 231.14 73.66 0)
+      (effects (font (size 1.27 1.27)))
+    )
+    (property "Footprint" "" (at 231.14 73.66 0)
+      (effects (font (size 1.27 1.27)) hide)
+    )
+    (property "Datasheet" "" (at 231.14 73.66 0)
+      (effects (font (size 1.27 1.27)) hide)
+    )
+    (pin "1A")
+    (pin "1B")
+    (pin "2A")
+    (pin "2B")
+    (pin "3A")
+    (pin "3B")
+    (pin "4A")
+    (pin "4B")
+    (instances
+      (project "NCNCA-Lap_Counter"
+        (path "/f7d7cc02-a4fd-4b7a-92a3-de67af0c24a1/981d6c09-cf16-465d-a2b6-16f1e2da1a1f"
+          (reference "TB1") (unit 1)
+        )
+      )
     )
   )
@@
         )
       )
-    )
-  )
-  (symbol (lib_id "Connector:Screw_Terminal_01x04") (at 229.87 83.82 90) (unit 1)
-    (in_bom yes) (on_board yes) (dnp no)
-    (property "Reference" "J1" (at 231.14 80.01 90)
-      (effects (font (size 1.27 1.27)))
-    )
-    (property "Value" "12V Terminal Block" (at 231.14 77.47 90)
-      (effects (font (size 1.27 1.27)))
-    )
-    (property "Footprint" "" (at 229.87 83.82 0)
-      (effects (font (size 1.27 1.27)) hide)
-    )
-    (property "Datasheet" "~" (at 229.87 83.82 0)
-      (effects (font (size 1.27 1.27)) hide)
-    )
-    (pin "1")
-    (pin "2")
-    (pin "3")
-    (pin "4")
-    (instances
-      (project "NCNCA-Lap_Counter"
-        (path "/f7d7cc02-a4fd-4b7a-92a3-de67af0c24a1/981d6c09-cf16-465d-a2b6-16f1e2da1a1f"
-          (reference "J1") (unit 1)
-        )
-      )

Commit message: schematic and pcb changes
Parts:
- removed BT1, BT2: 12V, symbol Device:Battery_Cell
- removed CR1: PowMr Charge Controller, symbol Project Library:PowMr
- removed DCC1: 12/24V to 5V Converter, symbol Project Library:PR4A065
- removed J2: Barrel_Jack, symbol Connector:Barrel_Jack
- removed J3: USB_A, symbol Connector:USB_A
- removed SC1: Solar_Cells, symbol Device:Solar_Cells
- removed SW1: SW_DPST_x2, symbol Switch:SW_DPST_x2
- removed TB1: ~, symbol Project Library:Terminal_Block_4
- added 1RM1: 1 Relay Module, symbol Project Library:1_Relay_Module
- added BT3: Battery 12v Li-ion, symbol Device:Battery
- added D1, D2: 1N4001, Diode_THT:D_DO-41_SOD81_P10.16mm_Horizontal, symbol Diode:1N4001
- added J1: Barrel_Jack, symbol Connector:Barrel_Jack
- added K1: RT424F12, Relay_THT:Relay_DPDT_Schrack-RT2-FormC-Dual-Coil_RM5mm, symbol Relay:RT42xFxx
- added SW2, SW3: SW_Push_SPDT, symbol Switch:SW_Push_SPDT
Connections:
- net 12V DC: now also K1.14
- net 5V DC: now also 1RM1.1 (DC+)
- net 5V GND: now also 1RM1.2 (DC-)
- new net: BT3.1 (+), D1.1 (K), D2.1 (K), J1.1, K1.11, K1.A3
- new net: D2.2 (A), K1.A1, SW3.3 (C)
- new net: 1RM1.6 (NO), D1.2 (A), K1.A2, SW2.3 (C)
- new net GND: 1RM1.5 (COM), BT3.2 (-), J1.2, SW2.2 (B), SW3.2 (B)
- new net PWR Disc: 1RM1.3 (IN)
- no-connect marks 2 -> 7
Other:
- note added: "CX"
- note added: "R1"
- note added: "S1"
- note added: "SALON Passive Bistable/Latching DPDT 8 Amp Power Relay Module, 12V Version, RT424F12"
- note added: "SX"
- note added: "V+"

Commit message: lots of diagram changes and software dir.
Parts:
- added VC1: ~, symbol Project Library:DC_12V_to_DC_5V_3A_Converter
Connections:
- net 12V DC: now also VC1.1 (12V+_In)
- net 5V DC: now also VC1.3 (5V+_Out)
- net GND: now also VC1.4 (GND_Out)
Changed lines of the file:
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@@
   (junction (at 226.06 147.32) (diameter 0) (color 0 0 0 0)
   )
+  (junction (at 314.96 157.48) (diameter 0) (color 0 0 0 0)
+  )
   (junction (at 246.38 147.32) (diameter 0) (color 0 0 0 0)
   )
   (junction (at 213.36 149.86) (diameter 0) (color 0 0 0 0)
   )
+  (junction (at 314.96 154.94) (diameter 0) (color 0 0 0 0)
+  )
   (junction (at 231.14 147.32) (diameter 0) (color 0 0 0 0)
   )
+  (junction (at 254 172.72) (diameter 0) (color 0 0 0 0)
+  )
+  (junction (at 281.94 154.94) (diameter 0) (color 0 0 0 0)
+  )
   (junction (at 238.76 147.32) (diameter 0) (color 0 0 0 0)
   )
@@
   )
   (junction (at 120.65 154.94) (diameter 0) (color 0 0 0 0)
+  )
+  (junction (at 281.94 157.48) (diameter 0) (color 0 0 0 0)
   )
   (no_connect (at 246.38 167.64))
@@
     (stroke (width 0) (type default))
   )
+  (wire (pts (xy 311.15 154.94) (xy 314.96 154.94))
+    (stroke (width 0) (type default))
+  )
   (wire (pts (xy 111.76 144.78) (xy 120.65 144.78))
     (stroke (width 0) (type default))
@@
     (stroke (width 0) (type default))
   )
+  (wire (pts (xy 254 172.72) (xy 256.54 172.72))
+    (stroke (width 0) (type default))
+  )
+  (wire (pts (xy 264.16 149.86) (xy 264.16 157.48))
+    (stroke (width 0) (type default))
+  )
+  (wire (pts (xy 281.94 154.94) (xy 254 154.94))
+    (stroke (width 0) (type default))
+  )
+  (wire (pts (xy 314.96 154.94) (xy 325.12 154.94))
+    (stroke (width 0) (type default))
+  )
+  (wire (pts (xy 264.16 157.48) (xy 281.94 157.48))
+    (stroke (width 0) (type default))
+  )
   (wire (pts (xy 223.52 147.32) (xy 226.06 147.32))
     (stroke (width 0) (type default))
   )
+  (wire (pts (xy 254 154.94) (xy 254 172.72))
+    (stroke (width 0) (type default))
+  )
+  (wire (pts (xy 314.96 157.48) (xy 325.12 157.48))
+    (stroke (width 0) (type default))
+  )
+  (wire (pts (xy 281.94 157.48) (xy 288.29 157.48))
+    (stroke (width 0) (type default))
+  )
   (wire (pts (xy 144.78 170.18) (xy 144.78 144.78))
     (stroke (width 0) (type default))
   )
+  (wire (pts (xy 288.29 154.94) (xy 281.94 154.94))
+    (stroke (width 0) (type default))
+  )
   (wire (pts (xy 226.06 139.7) (xy 194.31 139.7))
     (stroke (width 0) (type default))
   )
+  (wire (pts (xy 311.15 157.48) (xy 314.96 157.48))
+    (stroke (width 0) (type default))
+  )
   (wire (pts (xy 170.18 148.59) (xy 172.72 148.59))
     (stroke (width 0) (type default))
@@
     (stroke (width 0) (type default))
   )
-  (wire (pts (xy 246.38 172.72) (xy 256.54 172.72))
+  (wire (pts (xy 246.38 172.72) (xy 254 172.72))
     (stroke (width 0) (type default))
   )
@@
     )
   )
+  (global_label "5V DC" (shape passive) (at 325.12 154.94 0) (fields_autoplaced)
+    (effects (font (size 1.27 1.27)) (justify left))
+    (property "Intersheetrefs" "${INTERSHEET_REFS}" (at 332.7996 154.94 0)
+      (effects (font (size 1.27 1.27)) (justify left) hide)
+    )
+  )
   (global_label "12V GND" (shape passive) (at 210.82 149.86 180) (fields_autoplaced)
     (effects (font (size 1.27 1.27)) (justify right))
@@
     )
   )
+  (symbol (lib_id "power:PWR_FLAG") (at 314.96 157.48 0) (mirror x) (unit 1)
+    (in_bom yes) (on_board yes) (dnp no) (fields_autoplaced)
+    (property "Reference" "#FLG02" (at 314.96 159.385 0)
+      (effects (font (size 1.27 1.27)) hide)
+    )
+    (property "Value" "PWR_FLAG" (at 314.96 162.56 0)
+      (effects (font (size 1.27 1.27)))
+    )
+    (property "Footprint" "" (at 314.96 157.48 0)
+      (effects (font (size 1.27 1.27)) hide)
+    )
+    (property "Datasheet" "~" (at 314.96 157.48 0)
+      (effects (font (size 1.27 1.27)) hide)
+    )
+    (pin "1")
+    (instances
+      (project "NCNCA-Lap_Counter"
+        (path "/f7d7cc02-a4fd-4b7a-92a3-de67af0c24a1/981d6c09-cf16-465d-a2b6-16f1e2da1a1f"
+          (reference "#FLG02") (unit 1)
+        )
+      )
+    )
+  )
+  (symbol (lib_id "power:PWR_FLAG") (at 281.94 157.48 0) (mirror x) (unit 1)
+    (in_bom yes) (on_board yes) (dnp no) (fields_autoplaced)
+    (property "Reference" "#FLG04" (at 281.94 159.385 0)
+      (effects (font (size 1.27 1.27)) hide)
+    )
+    (property "Value" "PWR_FLAG" (at 281.94 162.56 0)
+      (effects (font (size 1.27 1.27)))
+    )
+    (property "Footprint" "" (at 281.94 157.48 0)
+      (effects (font (size 1.27 1.27)) hide)
+    )
+    (property "Datasheet" "~" (at 281.94 157.48 0)
+      (effects (font (size 1.27 1.27)) hide)
+    )
+    (pin "1")
+    (instances
+      (project "NCNCA-Lap_Counter"
+        (path "/f7d7cc02-a4fd-4b7a-92a3-de67af0c24a1/981d6c09-cf16-465d-a2b6-16f1e2da1a1f"
+          (reference "#FLG04") (unit 1)
+        )
+      )
+    )
+  )
   (symbol (lib_id "Connector:Barrel_Jack") (at 95.25 152.4 0) (unit 1)
     (in_bom yes) (on_board yes) (dnp no) (fields_autoplaced)
@@
         (path "/f7d7cc02-a4fd-4b7a-92a3-de67af0c24a1/981d6c09-cf16-465d-a2b6-16f1e2da1a1f"
           (reference "J1") (unit 1)
+        )
+      )
+    )
+  )
+  (symbol (lib_id "power:PWR_FLAG") (at 281.94 154.94 0) (unit 1)
+    (in_bom yes) (on_board yes) (dnp no) (fields_autoplaced)
+    (property "Reference" "#FLG03" (at 281.94 153.035 0)
+      (effects (font (size 1.27 1.27)) hide)
+    )
+    (property "Value" "PWR_FLAG" (at 281.94 149.86 0)
+      (effects (font (size 1.27 1.27)))
+    )
+    (property "Footprint" "" (at 281.94 154.94 0)
+      (effects (font (size 1.27 1.27)) hide)
+    )
+    (property "Datasheet" "~" (at 281.94 154.94 0)
+      (effects (font (size 1.27 1.27)) hide)
+    )
+    (pin "1")
+    (instances
+      (project "NCNCA-Lap_Counter"
+        (path "/f7d7cc02-a4fd-4b7a-92a3-de67af0c24a1/981d6c09-cf16-465d-a2b6-16f1e2da1a1f"
+          (reference "#FLG03") (unit 1)
         )
       )
@@
     )
   )
+  (symbol (lib_id "Project Library:DC_12V_to_DC_5V_3A_Converter") (at 299.72 151.13 0) (unit 1)
+    (in_bom yes) (on_board yes) (dnp no) (fields_autoplaced)
+    (property "Reference" "VC1" (at 299.72 149.86 0)
+      (effects (font (size 1.27 1.27)))
+    )
+    (property "Value" "~" (at 299.72 151.13 0)
+      (effects (font (size 1.27 1.27)))
+    )
+    (property "Footprint" "" (at 299.72 151.13 0)
+      (effects (font (size 1.27 1.27)) hide)
+    )
+    (property "Datasheet" "" (at 299.72 151.13 0)
+      (effects (font (size 1.27 1.27)) hide)
+    )
+    (pin "1")
+    (pin "2")
+    (pin "3")
+    (pin "4")
+    (instances
+      (project "NCNCA-Lap_Counter"
+        (path "/f7d7cc02-a4fd-4b7a-92a3-de67af0c24a1/981d6c09-cf16-465d-a2b6-16f1e2da1a1f"
+          (reference "VC1") (unit 1)
+        )
+      )
+    )
+  )
   (symbol (lib_id "Device:Battery") (at 120.65 149.86 0) (unit 1)
     (in_bom yes) (on_board yes) (dnp no) (fields_autoplaced)
@@
         (path "/f7d7cc02-a4fd-4b7a-92a3-de67af0c24a1/981d6c09-cf16-465d-a2b6-16f1e2da1a1f"
           (reference "SW3") (unit 1)
+        )
+      )
+    )
+  )
+  (symbol (lib_id "power:PWR_FLAG") (at 314.96 154.94 0) (unit 1)
+    (in_bom yes) (on_board yes) (dnp no) (fields_autoplaced)
+    (property "Reference" "#FLG01" (at 314.96 153.035 0)
+      (effects (font (size 1.27 1.27)) hide)
+    )
+    (property "Value" "PWR_FLAG" (at 314.96 149.86 0)
+      (effects (font (size 1.27 1.27)))
+    )
+    (property "Footprint" "" (at 314.96 154.94 0)
+      (effects (font (size 1.27 1.27)) hide)
+    )
+    (property "Datasheet" "~" (at 314.96 154.94 0)
+      (effects (font (size 1.27 1.27)) hide)
+    )
+    (pin "1")
+    (instances
+      (project "NCNCA-Lap_Counter"
+        (path "/f7d7cc02-a4fd-4b7a-92a3-de67af0c24a1/981d6c09-cf16-465d-a2b6-16f1e2da1a1f"
+          (reference "#FLG01") (unit 1)
         )
       )
@@
         )
       )
+    )
+  )
+  (symbol (lib_id "power:GND") (at 325.12 157.48 0) (unit 1)
+    (in_bom yes) (on_board yes) (dnp no) (fields_autoplaced)
+    (property "Reference" "#PWR03" (at 325.12 163.83 0)
+      (effects (font (size 1.27 1.27)) hide)
+    )
+    (property "Value" "GND" (at 325.12 162.56 0)
+      (effects (font (size 1.27 1.27)))
+    )
+    (property "Footprint" "" (at 325.12 157.48 0)
+      (effects (font (size 1.27 1.27)) hide)
+    )
+    (property "Datasheet" "" (at 325.12 157.48 0)
+      (effects (font (size 1.27 1.27)) hide)
+    )
+    (pin "1")
+    (instances
+      (project "NCNCA-Lap_Counter"
+        (path "/f7d7cc02-a4fd-4b7a-92a3-de67af0c24a1/981d6c09-cf16-465d-a2b6-16f1e2da1a1f"
+          (reference "#PWR03") (unit 1)
+        )
+      )
